Commit message: lab3 commit

File: dobot/urdf/dobot.xacro (robot description, xacro)
@@ -3,5 +3,5 @@
     <!-- Read from YAML -->
     <!-- Base -->
-    <xacro:property name="dobot" value="${xacro.load_yaml('$(find dobot)/config/params.yaml')}" />
+    <xacro:property name="dobot" value="${xacro.load_yaml('$(find dobot)/config/params.yaml').ForwardKin.ros__parameters}" />
     <xacro:property name="base_xy" value="${dobot.link_sizes.base.xy}" />
     <xacro:property name="base_z" value="${dobot.link_sizes.base.z}" />
